Commit message: Update newrobot.urdf

File: newrobot.urdf (robot description, URDF)
Before this commit: robot robot, 6 links, 5 joints
Joints:
- joint base_laser_horiz_joint: axis (none) -> 0 1 0
- joint base_laser_vert_bottom_joint: axis (none) -> 0 1 0
- joint base_laser_vert_top_left_joint: axis (none) -> 0 1 0
- joint base_laser_vert_top_right_joint: axis (none) -> 0 1 0
- joint base_wheel_left_joint: axis (none) -> 0 1 0

Commit message: Update newrobot.urdf

File: newrobot.urdf (robot description, URDF)
Before this commit: robot robot, 6 links, 5 joints
Joints:
- joint base_laser_horiz_joint: axis 0 1 0 -> (none)
- joint base_laser_vert_bottom_joint: axis 0 1 0 -> (none)
- joint base_laser_vert_top_left_joint: axis 0 1 0 -> (none)
- joint base_laser_vert_top_right_joint: axis 0 1 0 -> (none)
