Commit message: Update and rename robot.urdf to robot1.urdf

File: robot1.urdf (robot description, URDF)
Before this commit: robot robot, 6 links, 5 joints
Joints:
- joint base_wheel_left: axis (none) -> 0 1 0

Commit message: Update robot1.urdf

File: robot1.urdf (robot description, URDF)
Before this commit: robot robot1, 6 links, 5 joints
Joints:
- joint base_wheel_left: axis 0 1 0 -> (none)
